File: entradas.kicad_sch (KiCad schematic)
At the start: 10 parts, among them J5 BORNERA-2, J6 BORNERA-2, U4 TLP621, U5 TLP621

Commit message: avance en PCB y SCH
Parts:
- added D10, D9: LED, LED_SMD:LED_0805_2012Metric_Pad1.15x1.40mm_HandSolder, symbol Device:LED
- D5, D6: footprint Diode_SMD:D_MELF -> Diode_SMD:D_SMA_Handsoldering
Connections:
- net GND: now also D5.2 (A), D6.2 (A), U4.2, U5.2
- net at R11.1: now also J6.2 (Pin_2); no longer J6.1 (Pin_1)
- net at D6.1 (K), R11.2: now also D10.2 (A); no longer U5.1
- net at R9.1: now also J5.2 (Pin_2); no longer J5.1 (Pin_1)
- net at D5.1 (K), R9.2: now also D9.2 (A); no longer U4.1
- new net: D9.1 (K), U4.1
- new net: D10.1 (K), U5.1
- new net +VSW: J5.1 (Pin_1), J6.1 (Pin_1)
Other:
- moved on the sheet: D5, J5, J6, R8, R9, U4

Commit message: avance en PCB y SCH
Connections:
- net +VSW: now also J5.2 (Pin_2), J6.2 (Pin_2); no longer J5.1 (Pin_1), J6.1 (Pin_1)
- net at R11.1: now also J6.1 (Pin_1); no longer J6.2 (Pin_2)
- net at R9.1: now also J5.1 (Pin_1); no longer J5.2 (Pin_2)
Other:
- moved on the sheet: J5, J6
Changed lines of the file:
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@@
     (stroke (width 0) (type default) (color 0 0 0 0))
   )
-  (wire (pts (xy 118.11 107.95) (xy 118.11 105.41))
+  (wire (pts (xy 118.11 105.41) (xy 118.11 113.03))
     (stroke (width 0) (type default) (color 0 0 0 0))
   )
@@
     (stroke (width 0) (type default) (color 0 0 0 0))
   )
-  (wire (pts (xy 115.57 107.95) (xy 118.11 107.95))
-    (stroke (width 0) (type default) (color 0 0 0 0))
-  )
   (wire (pts (xy 147.32 120.65) (xy 134.62 120.65))
     (stroke (width 0) (type default) (color 0 0 0 0))
   )
-  (wire (pts (xy 116.84 59.69) (xy 116.84 57.15))
+  (wire (pts (xy 116.84 57.15) (xy 116.84 64.77))
     (stroke (width 0) (type default) (color 0 0 0 0))
   )
@@
     (stroke (width 0) (type default) (color 0 0 0 0))
   )
+  (wire (pts (xy 118.11 113.03) (xy 115.57 113.03))
+    (stroke (width 0) (type default) (color 0 0 0 0))
+  )
   (wire (pts (xy 165.1 115.57) (xy 165.1 120.65))
     (stroke (width 0) (type default) (color 0 0 0 0))
@@
     (stroke (width 0) (type default) (color 0 0 0 0))
   )
-  (wire (pts (xy 114.3 59.69) (xy 116.84 59.69))
-    (stroke (width 0) (type default) (color 0 0 0 0))
-  )
   (wire (pts (xy 130.81 110.49) (xy 134.62 110.49))
     (stroke (width 0) (type default) (color 0 0 0 0))
@@
   )
   (wire (pts (xy 163.83 67.31) (xy 163.83 72.39))
+    (stroke (width 0) (type default) (color 0 0 0 0))
+  )
+  (wire (pts (xy 116.84 64.77) (xy 114.3 64.77))
     (stroke (width 0) (type default) (color 0 0 0 0))
   )
@@
     (pin "2")
   )
-  (symbol (lib_id "Connector:Screw_Terminal_01x02") (at 109.22 59.69 0) (mirror y) (unit 1)
-    (in_bom yes) (on_board yes) (fields_autoplaced)
-    (property "Reference" "J5" (id 0) (at 109.22 53.34 0))
-    (property "Value" "BORNERA-2" (id 1) (at 109.22 55.88 0))
-    (property "Footprint" "TerminalBlock_Phoenix:TerminalBlock_Phoenix_MKDS-1,5-2-5.08_1x02_P5.08mm_Horizontal" (id 2) (at 109.22 59.69 0)
-      (effects (font (size 1.27 1.27)) hide)
-    )
-    (property "Datasheet" "~" (id 3) (at 109.22 59.69 0)
+  (symbol (lib_id "Connector:Screw_Terminal_01x02") (at 109.22 62.23 0) (mirror y) (unit 1)
+    (in_bom yes) (on_board yes) (fields_autoplaced)
+    (property "Reference" "J5" (id 0) (at 109.22 55.88 0))
+    (property "Value" "BORNERA-2" (id 1) (at 109.22 58.42 0))
+    (property "Footprint" "TerminalBlock_Phoenix:TerminalBlock_Phoenix_MKDS-1,5-2-5.08_1x02_P5.08mm_Horizontal" (id 2) (at 109.22 62.23 0)
+      (effects (font (size 1.27 1.27)) hide)
+    )
+    (property "Datasheet" "~" (id 3) (at 109.22 62.23 0)
       (effects (font (size 1.27 1.27)) hide)
     )
@@
     (pin "1")
   )
-  (symbol (lib_id "Connector:Screw_Terminal_01x02") (at 110.49 107.95 0) (mirror y) (unit 1)
-    (in_bom yes) (on_board yes) (fields_autoplaced)
-    (property "Reference" "J6" (id 0) (at 110.49 101.6 0))
-    (property "Value" "BORNERA-2" (id 1) (at 110.49 104.14 0))
-    (property "Footprint" "TerminalBlock_Phoenix:TerminalBlock_Phoenix_MKDS-1,5-2-5.08_1x02_P5.08mm_Horizontal" (id 2) (at 110.49 107.95 0)
-      (effects (font (size 1.27 1.27)) hide)
-    )
-    (property "Datasheet" "~" (id 3) (at 110.49 107.95 0)
-      (effects (font (size 1.27 1.27)) hide)
-    )
+  (symbol (lib_id "Connector:Screw_Terminal_01x02") (at 110.49 110.49 0) (mirror y) (unit 1)
+    (in_bom yes) (on_board yes) (fields_autoplaced)
+    (property "Reference" "J6" (id 0) (at 110.49 104.14 0))
+    (property "Value" "BORNERA-2" (id 1) (at 110.49 106.68 0))
+    (property "Footprint" "TerminalBlock_Phoenix:TerminalBlock_Phoenix_MKDS-1,5-2-5.08_1x02_P5.08mm_Horizontal" (id 2) (at 110.49 110.49 0)
+      (effects (font (size 1.27 1.27)) hide)
+    )
+    (property "Datasheet" "~" (id 3) (at 110.49 110.49 0)
+      (effects (font (size 1.27 1.27)) hide)
+    )
