File: salidas.kicad_sch (KiCad schematic)
At the start: 10 parts, among them J3 BORNERA-3, J4 BORNERA-3, K1 SANYOU_SRD_Form_C, K2 SANYOU_SRD_Form_C, Q1 2N7002K, Q2 2N7002K

Commit message: avance en PCB y SCH
Parts:
- added D7, D8: LED, LED_SMD:LED_0805_2012Metric_Pad1.15x1.40mm_HandSolder, symbol Device:LED
- added R12, R13: 1K, Resistor_SMD:R_0805_2012Metric_Pad1.20x1.40mm_HandSolder, symbol Device:R
- D3, D4: footprint Diode_SMD:D_MELF -> Diode_SMD:D_SMA_Handsoldering
- Q1, Q2: footprint Package_TO_SOT_SMD:SOT-23 -> Package_TO_SOT_SMD:SOT-23_Handsoldering
Connections:
- net +5V: now also R12.2, R13.2
- net at D3.2 (A), K1.2, Q1.3 (D): now also D7.1 (K)
- net at J4.1 (Pin_1): now also K2.3; no longer K2.4
- net at J4.3 (Pin_3): now also K2.4; no longer K2.3
- net at J3.1 (Pin_1): now also K1.3; no longer K1.4
- net at J3.3 (Pin_3): now also K1.4; no longer K1.3
- net at D4.2 (A), K2.2, Q2.3 (D): now also D8.1 (K)
- new net: D7.2 (A), R12.1
- new net: D8.2 (A), R13.1
Other:
- moved on the sheet: D3, J3, K1, Q1, R6

Commit message: avance en PCB y SCH
Connections:
- net +5V: now also D7.2 (A), D8.2 (A), K2.2; no longer K2.5, R12.2, R13.2
- net at D3.2 (A), K1.2, Q1.3 (D): now also R12.1; no longer D7.1 (K)
- net at J4.1 (Pin_1): now also K2.1; no longer K2.3
- net at J4.2 (Pin_2): now also K2.4; no longer K2.1
- net at J4.3 (Pin_3): now also K2.3; no longer K2.4
- net at J3.1 (Pin_1): now also K1.4; no longer K1.3
- net at J3.2 (Pin_2): now also K1.3; no longer K1.1
- net at J3.3 (Pin_3): now also K1.1; no longer K1.4
- net at D4.2 (A), Q2.3 (D): now also K2.5, R13.1; no longer D8.1 (K), K2.2
- new net: D7.1 (K), R12.2
- new net: D8.1 (K), R13.2
Other:
- moved on the sheet: D7, D8, J3, J4, K2, R12, R13
